File: adsr.kicad_sch (KiCad schematic)
At the start: 56 parts, among them J1 AudioJack2_SwitchT, J2 AudioJack2_SwitchT, J3 AudioJack2_SwitchT, J4 Conn_02x05_Odd_Even, Q1 BC547, Q2 BC547, Q3 BC547, Q4 BS170, SW1 SW_Push, SW2 SW_DPDT_x2, U1 ICM7555xB, U2 TL074

Commit message: first draft pcb
Parts:
- added H1: MountingHole, Eurorack:Mech-MountingHole, symbol Eurorack:MountingHole_Pad_Output
- added H10: trig, Eurorack:Mech-PushButton-Hole_Tayda_A-5051, symbol Mechanical:MountingHole_Pad
- added H11: out, Eurorack:Mech-AudioJack-Hole-Output, symbol Mechanical:MountingHole_Pad
- added H12: inv, Eurorack:Mech-AudioJack-Hole-Output, symbol Mechanical:MountingHole_Pad
- added H13: led, Eurorack:Mech-LED-Hole-4mm, symbol Mechanical:MountingHole_Pad
- added H14: speed, Eurorack:Mech-2M_Switch-Hole, symbol Mechanical:MountingHole_Pad
- added H2, H3, H4: MountingHole, Eurorack:Mech-MountingHole, symbol Mechanical:MountingHole_Pad
- added H5: attack, Eurorack:Mech-Potentiometer-Hole_level, symbol Mechanical:MountingHole_Pad
- added H6: decay, Eurorack:Mech-Potentiometer-Hole_level, symbol Mechanical:MountingHole_Pad
- added H7: sustain, Eurorack:Mech-Potentiometer-Hole_level, symbol Mechanical:MountingHole_Pad
- added H8: release, Eurorack:Mech-Potentiometer-Hole_level, symbol Mechanical:MountingHole_Pad
- added H9: gate, Eurorack:Mech-AudioJack-Hole, symbol Mechanical:MountingHole_Pad
- C1, C2, C4, C8: footprint (none) -> Capacitor_THT:CP_Radial_D5.0mm_P2.50mm
- C3, C5, C6, C7: footprint (none) -> Capacitor_SMD:C_0805_2012Metric
- D1, D2, D3, D4, D5: footprint (none) -> Diode_SMD:D_SOD-323_HandSoldering
- D6: footprint (none) -> LED_THT:LED_D3.0mm
- J1, J2, J3: footprint (none) -> Eurorack:AudioJack2_Tayda_A-2566
- J4: footprint (none) -> Eurorack:PinHeader_2x05_P2.54mm_Vertical
- JP1: footprint (none) -> Connector_PinHeader_2.54mm:PinHeader_1x02_P2.54mm_Vertical
- R1, R10, R11, R12, R13, R14, R15, R16, R17, R18, R19, R2, R20, R21, R22, R23, R3, R4, R5, R6, R7, R8, R9: footprint (none) -> Resistor_SMD:R_0805_2012Metric
- RV1, RV2, RV3, RV4: footprint (none) -> Eurorack:Potentiometer_RV16AF-41-15R1
- SW1: footprint (none) -> Eurorack:PushButton_Tayda_A-5051; PartNum (none) -> A-5051; Vendor (none) -> Tayda
- SW2: footprint (none) -> Eurorack:Switch_DPDT_Tayda_A-5752; PartNum (none) -> A-6809; Vendor (none) -> Tayda
- U2: footprint (none) -> Package_SO:SOIC-14_3.9x8.7mm_P1.27mm
Connections:
- net +12V: now also C7.1, D7.2 (K), D8.2 (K), U2.4 (V+); no longer R1.1
- net -12V: now also C7.2, D7.1 (A), D8.1 (A), U2.11 (V-); no longer R2.2
- net at Q4.3 (S), U1.7 (DIS): no longer RV4.1
- net at J4.10 (Pin_10), J4.9 (Pin_9): now also R2.1; no longer D8.3 (COM)
- net at J4.1 (Pin_1), J4.2 (Pin_2): now also R1.2; no longer D7.3 (COM)
- net at Q4.1 (D): now also RV4.1
- new net: D8.3 (COM), R2.2
- new net: D7.3 (COM), R1.1
- new net FACE: H1.1, H10.1, H11.1, H12.1, H13.1, H14.1, H2.1, H3.1, H4.1, H5.1, H6.1, H7.1, H8.1, H9.1
- no-connect marks 4 -> 7
Other:
- moved on the sheet: R1, R2

Commit message: slightly more compact pcb
Parts:
- Q1, Q2, Q3: footprint Package_TO_SOT_THT:TO-92_Inline -> Package_TO_SOT_THT:TO-92L_Inline_Wide
Changed lines of the file:
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@@
       (effects (font (size 1.27 1.27)) (justify left))
     )
-    (property "Footprint" "Package_TO_SOT_THT:TO-92_Inline" (at 123.19 85.725 0)
+    (property "Footprint" "Package_TO_SOT_THT:TO-92L_Inline_Wide" (at 123.19 85.725 0)
       (effects (font (size 1.27 1.27) italic) (justify left) hide)
     )
@@
       (effects (font (size 1.27 1.27)) (justify left))
     )
-    (property "Footprint" "Package_TO_SOT_THT:TO-92_Inline" (at 85.09 90.805 0)
+    (property "Footprint" "Package_TO_SOT_THT:TO-92L_Inline_Wide" (at 85.09 90.805 0)
       (effects (font (size 1.27 1.27) italic) (justify left) hide)
     )
@@
       (effects (font (size 1.27 1.27)) (justify left))
     )
-    (property "Footprint" "Package_TO_SOT_THT:TO-92_Inline" (at 64.77 90.805 0)
+    (property "Footprint" "Package_TO_SOT_THT:TO-92L_Inline_Wide" (at 64.77 90.805 0)
       (effects (font (size 1.27 1.27) italic) (justify left) hide)
     )

Commit message: removing non-parts from BOM
Parts:
- H10, H11, H12, H13, H14, H2, H3, H4, H5, H6, H7, H8, H9: now left out of the parts list
Changed lines of the file:
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@@
   )
   (symbol (lib_id "Mechanical:MountingHole_Pad") (at 90.17 140.97 0) (unit 1)
-    (in_bom yes) (on_board yes) (dnp no) (fields_autoplaced)
+    (in_bom no) (on_board yes) (dnp no) (fields_autoplaced)
     (property "Reference" "H12" (at 92.71 138.43 0)
       (effects (font (size 1.27 1.27)) (justify left))
@@
   )
   (symbol (lib_id "Mechanical:MountingHole_Pad") (at 90.17 128.27 0) (unit 1)
-    (in_bom yes) (on_board yes) (dnp no) (fields_autoplaced)
+    (in_bom no) (on_board yes) (dnp no) (fields_autoplaced)
     (property "Reference" "H10" (at 92.71 125.73 0)
       (effects (font (size 1.27 1.27)) (justify left))
@@
   )
   (symbol (lib_id "Mechanical:MountingHole_Pad") (at 90.17 121.92 0) (unit 1)
-    (in_bom yes) (on_board yes) (dnp no) (fields_autoplaced)
+    (in_bom no) (on_board yes) (dnp no) (fields_autoplaced)
     (property "Reference" "H9" (at 92.71 119.38 0)
       (effects (font (size 1.27 1.27)) (justify left))
@@
   )
   (symbol (lib_id "Mechanical:MountingHole_Pad") (at 54.61 128.27 0) (unit 1)
-    (in_bom yes) (on_board yes) (dnp no) (fields_autoplaced)
+    (in_bom no) (on_board yes) (dnp no) (fields_autoplaced)
     (property "Reference" "H2" (at 57.15 125.73 0)
       (effects (font (size 1.27 1.27)) (justify left))
@@
   )
   (symbol (lib_id "Mechanical:MountingHole_Pad") (at 74.93 121.92 0) (unit 1)
-    (in_bom yes) (on_board yes) (dnp no) (fields_autoplaced)
+    (in_bom no) (on_board yes) (dnp no) (fields_autoplaced)
     (property "Reference" "H5" (at 77.47 119.38 0)
       (effects (font (size 1.27 1.27)) (justify left))
@@
   )
   (symbol (lib_id "Mechanical:MountingHole_Pad") (at 54.61 134.62 0) (unit 1)
-    (in_bom yes) (on_board yes) (dnp no) (fields_autoplaced)
+    (in_bom no) (on_board yes) (dnp no) (fields_autoplaced)
     (property "Reference" "H3" (at 57.15 132.08 0)
       (effects (font (size 1.27 1.27)) (justify left))
@@
   )
   (symbol (lib_id "Mechanical:MountingHole_Pad") (at 90.17 134.62 0) (unit 1)
-    (in_bom yes) (on_board yes) (dnp no) (fields_autoplaced)
+    (in_bom no) (on_board yes) (dnp no) (fields_autoplaced)
     (property "Reference" "H11" (at 92.71 132.08 0)
       (effects (font (size 1.27 1.27)) (justify left))
@@
   )
   (symbol (lib_id "Mechanical:MountingHole_Pad") (at 101.6 121.92 0) (unit 1)
-    (in_bom yes) (on_board yes) (dnp no) (fields_autoplaced)
+    (in_bom no) (on_board yes) (dnp no) (fields_autoplaced)
     (property "Reference" "H13" (at 104.14 119.38 0)
       (effects (font (size 1.27 1.27)) (justify left))
@@
   )
   (symbol (lib_id "Mechanical:MountingHole_Pad") (at 54.61 140.97 0) (unit 1)
-    (in_bom yes) (on_board yes) (dnp no) (fields_autoplaced)
+    (in_bom no) (on_board yes) (dnp no) (fields_autoplaced)
     (property "Reference" "H4" (at 57.15 138.43 0)
       (effects (font (size 1.27 1.27)) (justify left))
@@
   )
   (symbol (lib_id "Mechanical:MountingHole_Pad") (at 74.93 134.62 0) (unit 1)
-    (in_bom yes) (on_board yes) (dnp no) (fields_autoplaced)
+    (in_bom no) (on_board yes) (dnp no) (fields_autoplaced)
     (property "Reference" "H7" (at 77.47 132.08 0)
       (effects (font (size 1.27 1.27)) (justify left))
@@
   )
   (symbol (lib_id "Mechanical:MountingHole_Pad") (at 74.93 128.27 0) (unit 1)
-    (in_bom yes) (on_board yes) (dnp no) (fields_autoplaced)
+    (in_bom no) (on_board yes) (dnp no) (fields_autoplaced)
     (property "Reference" "H6" (at 77.47 125.73 0)
       (effects (font (size 1.27 1.27)) (justify left))
@@
   )
   (symbol (lib_id "Mechanical:MountingHole_Pad") (at 101.6 128.27 0) (unit 1)
-    (in_bom yes) (on_board yes) (dnp no) (fields_autoplaced)
+    (in_bom no) (on_board yes) (dnp no) (fields_autoplaced)
     (property "Reference" "H14" (at 104.14 125.73 0)
       (effects (font (size 1.27 1.27)) (justify left))
@@
   )
   (symbol (lib_id "Mechanical:MountingHole_Pad") (at 74.93 140.97 0) (unit 1)
-    (in_bom yes) (on_board yes) (dnp no) (fields_autoplaced)
+    (in_bom no) (on_board yes) (dnp no) (fields_autoplaced)
     (property "Reference" "H8" (at 77.47 138.43 0)
       (effects (font (size 1.27 1.27)) (justify left))

Commit message: v2 fixes
Parts:
- C4, C8: symbol Device:C -> Device:C_Polarized
- H13: footprint Eurorack:Mech-LED-Hole-4mm -> Eurorack:Mech-LED-Hole-3mm-Bezel
- Q1, Q2, Q3: PartNum 771-BCM847DS135 -> 637-BC547C
Connections:
- net GND: now also C4.2, C8.2; no longer C4.1, C8.1
- net SUSTAIN: now also U2.10 (+); no longer U2.9 (-)
- net at RV2.1: now also D4.2 (A)
- net at SW2.4 (A): now also C8.1; no longer C8.2
- net at D4.1 (K), U2.8: now also U2.9 (-); no longer U2.10 (+)
- net at SW2.6 (C): now also C4.1; no longer C4.2
- net DECAY_CW: no longer names the net of RV2.3
- net DECAY_CW: no longer D4.2 (A)
Other:
- moved on the sheet: C6, D2, D3, D4, R16, R17, R20, RV2, RV4, U2C

Commit message: updating BOM for v2
Parts:
- C1, C2: value 22u 35V -> 22u 50V
- C8: value 1u 35V Tant -> 1u 50V Tant
Changed lines of the file:
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@@
       (effects (font (size 1.27 1.27)) (justify right))
     )
-    (property "Value" "1u 35V Tant" (at 226.06 98.171 0)
+    (property "Value" "1u 50V Tant" (at 226.06 98.171 0)
       (effects (font (size 1.27 1.27)) (justify right))
     )
@@
       (effects (font (size 1.27 1.27)) (justify left))
     )
-    (property "Value" "22u 35V" (at 128.27 165.1 0)
+    (property "Value" "22u 50V" (at 128.27 165.1 0)
       (effects (font (size 1.27 1.27)) (justify left))
     )
@@
       (effects (font (size 1.27 1.27)) (justify left))
     )
-    (property "Value" "22u 35V" (at 128.27 181.61 0)
-      (effects (font (size 1.27 1.27)) (justify left))
-    )
+    (property "Value" "22u 50V" (at 128.27 181.61 0)
+      (effects (font (size 1.27 1.27)) (justify left))
+    )

Commit message: new design language, adding pcb to readme
Parts:
- H11, H12: footprint Eurorack:Mech-AudioJack-Hole-Output -> Eurorack:Mech-AudioJack-Hole-Output-CV
- H9: footprint Eurorack:Mech-AudioJack-Hole -> Eurorack:Mech-AudioJack-Hole-Input-Gate
Changed lines of the file:
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@@
       (effects (font (size 1.27 1.27)) (justify left))
     )
-    (property "Footprint" "Eurorack:Mech-AudioJack-Hole-Output" (at 90.17 140.97 0)
+    (property "Footprint" "Eurorack:Mech-AudioJack-Hole-Output-CV" (at 90.17 140.97 0)
       (effects (font (size 1.27 1.27)) hide)
     )
@@
       (effects (font (size 1.27 1.27)) (justify left))
     )
-    (property "Footprint" "Eurorack:Mech-AudioJack-Hole" (at 90.17 121.92 0)
+    (property "Footprint" "Eurorack:Mech-AudioJack-Hole-Input-Gate" (at 90.17 121.92 0)
       (effects (font (size 1.27 1.27)) hide)
     )
@@
       (effects (font (size 1.27 1.27)) (justify left))
     )
-    (property "Footprint" "Eurorack:Mech-AudioJack-Hole-Output" (at 90.17 134.62 0)
-      (effects (font (size 1.27 1.27)) hide)
-    )
+    (property "Footprint" "Eurorack:Mech-AudioJack-Hole-Output-CV" (at 90.17 134.62 0)
+      (effects (font (size 1.27 1.27)) hide)
+    )
